File: hardware/tube_board/tube_board.brd (EAGLE design)
At the start: 125 x 30 mm, 27 parts, among them IC2 TPS77333, K1 651005136421, Q1 16MHz

Commit message: Finish schematic and start board layout
Parts:
- removed C11: 0.1uF, resistor:C0603
- removed R4: 10k, rcl:R0603
- removed U$1: MC33063/MC34063D, adafruit:SO08
- added C10: 4.7uF, resistor:C0603
- added C12, C13: EEE-1VA221UP, rcl:PANASONIC_G
- added C14: 0.01uF, resistor:C0603
- added C15: 2200pF, resistor:C0603
- added C7: 1uF, resistor:C0603
- added C8: 47nF, resistor:C0603
- added C9: 33pF, resistor:C0603
- added D2: 1N914, diode:SOD323-R
- added D3: BAV21, diode:DO35-10
- added IC1: TPS61081, texas:S-PDSO-N10
- added L1: VLCF5020T-4R7N1R7-1, rcl:L5650M
- added L2: DRA127-221-R, inductors:DR127
- added LED1, LED2, LED3, LED4, LED5, LED6, LED7, LED8: (no value), led:CHIPLED_0603
- added Q2: IRF740, transistor-power:TO220BV
- added Q3: MPSA56, transistor-pnp:TO92-CBE
- added Q4: (no value), adafruit:SOT23
- added R10: 100, rcl:R0603
- added R11, R12, R13, R14, R15, R16, R17, R18, R19, R20, R6: 1k, rcl:R0603
- added R8: 437k, rcl:R0603
- added R9: 49.9k, rcl:R0603
- added TP1: TPTP07R, testpad:TP07R
- added U$6: MC34063D, adafruit:SO08
- N1, N2, N3, N4: value IN-14 -> IN-14SMD; device russian-nixies:IN-14 -> russian-nixies:IN-14-SMD
- moved IC2 322.9 mm to (149.0, 66.0), flipped to the bottom
- moved R5 313.9 mm to (127.0, 68.0), flipped to the bottom
- moved U$3 292.8 mm to (148.0, 41.0), flipped to the bottom
- moved R7 289.2 mm to (83.0, 80.0), flipped to the bottom
- moved C6 277.2 mm to (130.0, 52.0), flipped to the bottom
- moved R3 268.3 mm to (116.0, 60.0), flipped to the bottom
- moved D1 237.2 mm to (119.0, 14.0)
- moved R2 170.1 mm to (65.0, 61.0), flipped to the bottom
- moved JP2 169.3 mm to (62.0, 3.00), flipped to the bottom
- moved C4 169.2 mm to (75.0, 56.0), flipped to the bottom
- moved C1 152.6 mm to (72.0, 44.0), flipped to the bottom
- moved C3 149.9 mm to (63.0, 53.0), flipped to the bottom
- moved C5 149.3 mm to (59.0, 39.0), flipped to the bottom
- moved Q1 145.0 mm to (68.0, 27.0), flipped to the bottom, turned to 180 degrees
- moved R1 143.7 mm to (62.0, 47.0), flipped to the bottom
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Connections:
- removed net NIXIE_PWM: U$2.12
- removed net VCC: U$1.6
- removed net VDD: U$4.30, U$5.30
- removed net VSS: U$4.29, U$5.29
- new net +12V: C10.1, C12.+, C9.1, IC1.9, L2.2, R8.1, U$4.30, U$5.27, U$5.30, U$6.1, U$6.6, U$6.7, U$6.8
- new net 12V_EN: IC1.6, U$2.29
- new net DIGIT0_0: N1.0, U$4.22
- new net DIGIT0_1: N1.1, U$4.21
- new net DIGIT0_2: N1.2, U$4.20
- new net DIGIT0_3: N1.3, U$4.19
- new net DIGIT0_4: N1.4, U$4.18
- new net DIGIT0_5: N1.5, U$4.17
- new net DIGIT0_6: N1.6, U$4.16
- new net DIGIT0_7: N1.7, U$4.15
- new net DIGIT0_8: N1.8, U$4.14
- new net DIGIT0_9: N1.9, U$4.13
- new net DIGIT0_LD: N1.LHDP, U$4.11
- new net DIGIT0_RD: N1.RHDP, U$4.12
- new net DIGIT1_0: N2.0, U$4.3
- new net DIGIT1_1: N2.1, U$4.2
- new net DIGIT1_2: N2.2, U$4.1
- new net DIGIT1_3: N2.3, U$4.44
- new net DIGIT1_4: N2.4, U$4.43
- new net DIGIT1_5: N2.5, U$4.42
- new net DIGIT1_6: N2.6, U$4.41
- new net DIGIT1_7: N2.7, U$4.40
- new net DIGIT1_8: N2.8, U$4.39
- new net DIGIT1_9: N2.9, U$4.38
- new net DIGIT1_LD: N2.LHDP, U$4.36
- new net DIGIT1_RD: N2.RHDP, U$4.37
- new net DIGIT2_0: N3.0, U$5.22
- new net DIGIT2_1: N3.1, U$5.21
- new net DIGIT2_2: N3.2, U$5.20
- new net DIGIT2_3: N3.3, U$5.19
- new net DIGIT2_4: N3.4, U$5.18
- new net DIGIT2_5: N3.5, U$5.17
- new net DIGIT2_6: N3.6, U$5.16
- new net DIGIT2_7: N3.7, U$5.15
- new net DIGIT2_8: N3.8, U$5.14
- new net DIGIT2_9: N3.9, U$5.13
- new net DIGIT2_LD: N3.LHDP, U$5.11
- new net DIGIT2_RD: N3.RHDP, U$5.12
- new net DIGIT3_0: N4.0, U$5.3
- new net DIGIT3_1: N4.1, U$5.2
- new net DIGIT3_2: N4.2, U$5.1
- new net DIGIT3_3: N4.3, U$5.44
- new net DIGIT3_4: N4.4, U$5.43
- new net DIGIT3_5: N4.5, U$5.42
- new net DIGIT3_6: N4.6, U$5.41
- new net DIGIT3_7: N4.7, U$5.40
- new net DIGIT3_8: N4.8, U$5.39
- new net DIGIT3_9: N4.9, U$5.38
- new net DIGIT3_LD: N4.LHDP, U$5.36
- new net DIGIT3_RD: N4.RHDP, U$5.37
- new net HV_BLANK: U$2.12, U$4.33, U$5.33
- new net HV_FB: C14.1, R12.2, R13.1, U$6.5
- new net HV_LOAD: U$2.28, U$4.31, U$5.31
- new net HV_SHIFT: U$4.23, U$5.32
- new net N$10: C8.1, IC1.3
- new net N$11: D2.A, Q3.B, R11.1, U$6.2
- new net N$12: C9.2, R10.1, R8.2, R9.1
- new net N$13: D3.A, L2.1, Q2.D
- new net N$14: C15.1, U$6.3
- new net N$15: IC1.5, R10.2
- new net N$16: D2.C, Q2.G, Q3.E
- new net N$17: LED1.A, R6.2
- new net N$18: LED2.A, R14.2
- new net N$19: LED3.A, R15.2
- new net N$20: LED4.A, R16.2
- new net N$21: LED5.A, R17.2
- new net N$22: LED6.A, R18.2
- new net N$23: LED7.A, R19.2
- new net N$24: LED8.A, R20.2
- new net N$25: LED1.C, LED2.C, LED3.C, LED4.C, LED5.C, LED6.C, LED7.C, LED8.C, Q4.3
- new net N$31: U$4.27
- new net N$40: TP1.TP, U$5.23
- new net N$8: IC1.1, L1.1
- new net N$9: IC1.10, L1.2
- new net V+: C13.+, D3.C, N1.A, N2.A, N3.A, N4.A, R12.1
- net +5V: now also C7.1, IC1.2, IC1.7, R14.1, R15.1, R16.1, R17.1, R18.1, R19.1, R20.1, R6.1
- net GND: now also C10.2, C12.-, C13.-, C14.2, C15.2, C7.2, C8.2, IC1.4, IC1.8, Q2.S, Q3.C, Q4.2, R11.2, R13.2, R9.2, U$4.29, U$5.29, U$6.4; no longer U$1.4
- net LED_PWM: now also Q4.1
- net SPI0_MOSI: now also U$4.32
- net SPI0_SCLK: now also U$4.28, U$5.28

Commit message: WIP board layout
Parts:
- moved L1 97.1 mm to (21.0, 5.00), flipped to the top
- moved C12 79.6 mm to (24.0, 69.0), flipped to the top
- moved IC1 78.2 mm to (10.0, 16.0), flipped to the top, turned to 90 degrees
- moved C13 52.3 mm to (8.00, 76.0), flipped to the top
- moved U$2 38.3 mm to (90.0, 47.0), flipped to the top
- moved U$5 30.5 mm to (112.0, 43.0), flipped to the top
- moved U$4 29.0 mm to (46.0, 44.0), flipped to the top
- moved L2 18.8 mm to (22.0, 40.0), flipped to the top
- moved K1 3.00 mm to (3.00, 18.0), flipped to the top
- flipped C1 to the top
- flipped C10 to the top
- flipped C14 to the top
- flipped C15 to the top
- flipped C3 to the top
- flipped C4 to the top
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
Commit message: Hacky autorouted board
Parts:
- removed D3: BAV21, diode:DO35-10
- removed Q3: MPSA56, transistor-pnp:TO92-CBE
- D2: value 1N914 -> BAV21
- moved C7 149.4 mm to (5.00, 11.0), turned to 180 degrees
- moved IC2 142.2 mm to (21.0, 4.00), turned to 90 degrees
- moved C14 125.3 mm to (15.0, 19.0)
- moved R11 120.2 mm to (17.0, 26.0), turned to 270 degrees
- moved R5 119.4 mm to (27.0, 2.75), turned to 270 degrees
- moved C8 118.9 mm to (14.0, 9.00), turned to 270 degrees
- moved R13 118.0 mm to (17.0, 21.0)
- moved C15 117.5 mm to (10.0, 22.0), turned to 180 degrees
- moved D2 117.4 mm to (21.0, 23.0)
- moved R12 116.3 mm to (17.0, 23.0), turned to 180 degrees
- moved R8 113.9 mm to (10.0, 14.0)
- moved Q2 109.2 mm to (24.0, 29.0)
- moved C10 109.0 mm to (5.00, 9.00), turned to 180 degrees
- moved R9 106.8 mm to (16.0, 13.0), turned to 270 degrees
- moved R10 104.9 mm to (14.0, 13.0), turned to 270 degrees
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Connections:
- removed net N$11: D2.A, Q3.B, R11.1, U$6.2
- net GND: no longer Q3.C
- net N$13: now also D2.A; no longer D3.A
- net N$16: now also R11.1, U$6.2; no longer D2.C, Q3.E
- net V+: now also D2.C; no longer D3.C
Routing:
- net +5V: track 0.00 -> 259.2 mm, vias 0 -> 11
- net +12V: track 0.00 -> 183.6 mm, vias 0 -> 12
- net V+: track 0.00 -> 129.1 mm, vias 0 -> 11
- net N$25: track 0.00 -> 125.9 mm, vias 0 -> 10
- net USB_D+: track 0.00 -> 90.9 mm, vias 0 -> 4
- net SPI0_SCLK: track 0.00 -> 78.2 mm, vias 0 -> 11
- net DIGIT2_6: track 0.00 -> 73.6 mm, vias 0 -> 3
- net DIGIT0_8: track 0.00 -> 70.5 mm, vias 0 -> 1
- net DIGIT0_LD: track 0.00 -> 66.5 mm, vias 0 -> 3
- net HV_LOAD: track 0.00 -> 65.5 mm, vias 0 -> 4
- net DIGIT2_9: track 0.00 -> 61.9 mm, vias 0 -> 5
- net DIGIT0_9: track 0.00 -> 59.8 mm, vias 0 -> 3
- net DIGIT0_5: track 0.00 -> 50.8 mm, vias 0 -> 5
- net DIGIT2_7: track 0.00 -> 50.5 mm, vias 0 -> 5
- net DIGIT0_4: track 0.00 -> 49.0 mm, vias 0 -> 3
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- added copper zone on layer 1, net GND
- added copper zone on layer 16, net GND
Other:
- board size 125 x 30 mm -> 125 x 32 mm
