File: hardware/tube_board/tube_board.sch (EAGLE design)
At the start: 27 parts, among them IC2 TPS77333, K1 651005136421, Q1 16MHz

Commit message: Finish schematic and start board layout
Parts:
- removed C11: 0.1uF, resistor:C-USC0603
- removed R4: 10k, rcl:R-US_R0603
- removed U$1: MC33063/MC34063D, adafruit:MC33063/MC34063D
- added C10: 4.7uF, resistor:C-USC0603
- added C12, C13: EEE-1VA221UP, rcl:CPOL-USG
- added C14: 0.01uF, resistor:C-USC0603
- added C15: 2200pF, resistor:C-USC0603
- added C7: 1uF, resistor:C-USC0603
- added C8: 47nF, resistor:C-USC0603
- added C9: 33pF, resistor:C-USC0603
- added D2: 1N914, diode:DIODE-SOD323-R
- added D3: BAV21, diode:BAV21
- added IC1: TPS61081, texas:TPS61081
- added L1: VLCF5020T-4R7N1R7-1, rcl:L-USL5650M
- added L2: DRA127-221-R, inductors:DR127
- added LED1, LED2, LED3, LED4, LED5, LED6, LED7, LED8: (no value), led:LEDCHIPLED_0603
- added Q2: IRF740, transistor-power:IRF740
- added Q3: MPSA56, transistor-pnp:MPSA56
- added Q4: (no value), adafruit:MOSFET-NREFLOW
- added R10: 100, rcl:R-US_R0603
- added R11, R12, R13, R14, R15, R16, R17, R18, R19, R20, R6: 1k, rcl:R-US_R0603
- added R8: 437k, rcl:R-US_R0603
- added R9: 49.9k, rcl:R-US_R0603
- added TP1: TPTP07R, testpad:TPTP07R
- added U$6: MC34063D, adafruit:MC33063/MC34063D
- N1, N2, N3, N4: value IN-14 -> IN-14SMD; device russian-nixies:IN-14 -> russian-nixies:IN-14SMD
Connections:
- removed net NIXIE_PWM: U$2.PB7(OC0A/OC1C/RTS)
- new net +12V: C10.1, C12.+, C9.1, IC1G$1.OUT, L2.2, R8.1, U$4.VDD, U$5.VDD, U$5._POL, U$6.DC, U$6.IPK, U$6.SWC, U$6.VCC
- new net 12V_EN: IC1G$1.EN, U$2.PB5(OC1A/ADC12/!OC4B)
- new net DIGIT0_0: N1.0, U$4.HVOUT_1
- new net DIGIT0_1: N1.1, U$4.HVOUT_2
- new net DIGIT0_2: N1.2, U$4.HVOUT_3
- new net DIGIT0_3: N1.3, U$4.HVOUT_4
- new net DIGIT0_4: N1.4, U$4.HVOUT_5
- new net DIGIT0_5: N1.5, U$4.HVOUT_6
- new net DIGIT0_6: N1.6, U$4.HVOUT_7
- new net DIGIT0_7: N1.7, U$4.HVOUT_8
- new net DIGIT0_8: N1.8, U$4.HVOUT_9
- new net DIGIT0_9: N1.9, U$4.HVOUT_10
- new net DIGIT0_LD: N1.LHDP, U$4.HVOUT_12
- new net DIGIT0_RD: N1.RHDP, U$4.HVOUT_11
- new net DIGIT1_0: N2.0, U$4.HVOUT_20
- new net DIGIT1_1: N2.1, U$4.HVOUT_21
- new net DIGIT1_2: N2.2, U$4.HVOUT_22
- new net DIGIT1_3: N2.3, U$4.HVOUT_23
- new net DIGIT1_4: N2.4, U$4.HVOUT_24
- new net DIGIT1_5: N2.5, U$4.HVOUT_25
- new net DIGIT1_6: N2.6, U$4.HVOUT_26
- new net DIGIT1_7: N2.7, U$4.HVOUT_27
- new net DIGIT1_8: N2.8, U$4.HVOUT_28
- new net DIGIT1_9: N2.9, U$4.HVOUT_29
- new net DIGIT1_LD: N2.LHDP, U$4.HVOUT_31
- new net DIGIT1_RD: N2.RHDP, U$4.HVOUT_30
- new net DIGIT2_0: N3.0, U$5.HVOUT_1
- new net DIGIT2_1: N3.1, U$5.HVOUT_2
- new net DIGIT2_2: N3.2, U$5.HVOUT_3
- new net DIGIT2_3: N3.3, U$5.HVOUT_4
- new net DIGIT2_4: N3.4, U$5.HVOUT_5
- new net DIGIT2_5: N3.5, U$5.HVOUT_6
- new net DIGIT2_6: N3.6, U$5.HVOUT_7
- new net DIGIT2_7: N3.7, U$5.HVOUT_8
- new net DIGIT2_8: N3.8, U$5.HVOUT_9
- new net DIGIT2_9: N3.9, U$5.HVOUT_10
- new net DIGIT2_LD: N3.LHDP, U$5.HVOUT_12
- new net DIGIT2_RD: N3.RHDP, U$5.HVOUT_11
- new net DIGIT3_0: N4.0, U$5.HVOUT_20
- new net DIGIT3_1: N4.1, U$5.HVOUT_21
- new net DIGIT3_2: N4.2, U$5.HVOUT_22
- new net DIGIT3_3: N4.3, U$5.HVOUT_23
- new net DIGIT3_4: N4.4, U$5.HVOUT_24
- new net DIGIT3_5: N4.5, U$5.HVOUT_25
- new net DIGIT3_6: N4.6, U$5.HVOUT_26
- new net DIGIT3_7: N4.7, U$5.HVOUT_27
- new net DIGIT3_8: N4.8, U$5.HVOUT_28
- new net DIGIT3_9: N4.9, U$5.HVOUT_29
- new net DIGIT3_LD: N4.LHDP, U$5.HVOUT_31
- new net DIGIT3_RD: N4.RHDP, U$5.HVOUT_30
- new net HV_BLANK: U$2.PB7(OC0A/OC1C/RTS), U$4._BLANK, U$5._BLANK
- new net HV_FB: C14.1, R12.2, R13.1, U$6.COMP
- new net HV_LOAD: U$2.PB4(ADC11), U$4._LE, U$5._LE
- new net HV_SHIFT: U$4.DATAOUT, U$5.DATAIN
- new net N$10: C8.1, IC1G$1.SS
- new net N$11: D2.A, Q3.B, R11.1, U$6.SWE
- new net N$12: C9.2, R10.1, R8.2, R9.1
- new net N$13: D3.A, L2.1, Q2.D
- new net N$14: C15.1, U$6.TC
- new net N$15: IC1G$1.FB, R10.2
- new net N$16: D2.C, Q2.G, Q3.E
- new net N$17: LED1.A, R6.2
- new net N$18: LED2.A, R14.2
- new net N$19: LED3.A, R15.2
- new net N$20: LED4.A, R16.2
- new net N$21: LED5.A, R17.2
- new net N$22: LED6.A, R18.2
- new net N$23: LED7.A, R19.2
- new net N$24: LED8.A, R20.2
- new net N$25: LED1.C, LED2.C, LED3.C, LED4.C, LED5.C, LED6.C, LED7.C, LED8.C, Q4.D
- new net N$31: U$4._POL
- new net N$40: TP1.TP, U$5.DATAOUT
- new net N$8: IC1G$1.L, L1.1
- new net N$9: IC1G$1.SW, L1.2
- new net V+: C13.+, D3.C, N1.A, N2.A, N3.A, N4.A, R12.1
- net +5V: now also C7.1, IC1G$1.FSW, IC1G$1.VIN, R14.1, R15.1, R16.1, R17.1, R18.1, R19.1, R20.1, R6.1
- net GND: now also C10.2, C12.-, C13.-, C14.2, C15.2, C7.2, C8.2, IC1G$1.GND, IC1G$1.PGND, Q2.S, Q3.C, Q4.S, R11.2, R13.2, R9.2, U$4.VSS, U$5.VSS, U$6.GND
- net LED_PWM: now also Q4.G
- net SPI0_MOSI: now also U$4.DATAIN
- net SPI0_SCLK: now also U$4.CLK, U$5.CLK
Other:
- note added: "1. Power Supply 2. Micro 3. Tubes"
- note added: "12V to 180V"
- note added: "5V to 12V"
- note added: "Copied from TI datasheet"
- note added: "Power Supplies"
- note added: "Shamelessly copied from https://threeneurons.wordpress.com/nixie-power-supply/"
- note added: "Tubes and Drivers"
- note removed: "1. Tubes"
- note removed: "Tubes and Connectors"

Commit message: Hacky autorouted board
Parts:
- removed D3: BAV21, diode:BAV21
- removed Q3: MPSA56, transistor-pnp:MPSA56
- D2: value 1N914 -> BAV21
Connections:
- removed net N$11: D2.A, Q3.B, R11.1, U$6.SWE
- net GND: no longer Q3.C
- net N$13: now also D2.A; no longer D3.A
- net N$16: now also R11.1, U$6.SWE; no longer D2.C, Q3.E
- net V+: now also D2.C; no longer D3.C
Other:
- moved on the sheet: D2
Changed lines of the file:
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@@
 <?xml version="1.0" encoding="utf-8"?>
 <!DOCTYPE eagle SYSTEM "eagle.dtd">
-<eagle version="7.7.0">
+<eagle version="8.1.0">
 <drawing>
 <settings>
@@
 <layer number="2" name="Route2" color="1" fill="3" visible="yes" active="no"/>
 <layer number="3" name="Route3" color="4" fill="3" visible="yes" active="no"/>
+<layer number="4" name="Route4" color="1" fill="4" visible="no" active="no"/>
+<layer number="5" name="Route5" color="4" fill="4" visible="no" active="no"/>
+<layer number="6" name="Route6" color="1" fill="8" visible="no" active="no"/>
+<layer number="7" name="Route7" color="4" fill="8" visible="no" active="no"/>
+<layer number="8" name="Route8" color="1" fill="2" visible="no" active="no"/>
+<layer number="9" name="Route9" color="4" fill="2" visible="no" active="no"/>
+<layer number="10" name="Route10" color="1" fill="7" visible="no" active="no"/>
+<layer number="11" name="Route11" color="4" fill="7" visible="no" active="no"/>
+<layer number="12" name="Route12" color="1" fill="5" visible="no" active="no"/>
+<layer number="13" name="Route13" color="4" fill="5" visible="no" active="no"/>
 <layer number="14" name="Route14" color="1" fill="6" visible="yes" active="no"/>
 <layer number="15" name="Route15" color="4" fill="6" visible="yes" active="no"/>
@@
 <part name="Q2" library="transistor-power" deviceset="IRF740" device=""/>
 <part name="GND23" library="supply1" deviceset="GND" device=""/>
-<part name="Q3" library="transistor-pnp" deviceset="MPSA56*" device=""/>
-<part name="D2" library="diode" deviceset="DIODE-" device="SOD323-R" value="1N914"/>
 <part name="R11" library="rcl" deviceset="R-US_" device="R0603" value="1k"/>
 <part name="GND24" library="supply1" deviceset="GND" device=""/>
-<part name="GND25" library="supply1" deviceset="GND" device=""/>
-<part name="D3" library="diode" deviceset="BAV21" device=""/>
 <part name="C13" library="rcl" deviceset="CPOL-US" device="G" value="EEE-1VA221UP"/>
 <part name="GND26" library="supply1" deviceset="GND" device=""/>
@@
 <part name="SUPPLY4" library="supply2" deviceset="V+" device=""/>
 <part name="SUPPLY5" library="supply2" deviceset="V+" device=""/>
+<part name="D2" library="diode" deviceset="DIODE-" device="SOD323-R" value="BAV21"/>
 </parts>
 <sheets>
@@
 <instance part="Q2" gate="G$1" x="111.76" y="86.36"/>
 <instance part="GND23" gate="1" x="114.3" y="60.96"/>
-<instance part="Q3" gate="G$1" x="129.54" y="71.12"/>
-<instance part="D2" gate="G$1" x="137.16" y="81.28" rot="R180"/>
 <instance part="R11" gate="G$1" x="144.78" y="71.12" rot="R270"/>
 <instance part="GND24" gate="1" x="144.78" y="60.96"/>
-<instance part="GND25" gate="1" x="132.08" y="60.96"/>
-<instance part="D3" gate="1" x="104.14" y="93.98" rot="R180"/>
 <instance part="C13" gate="G$1" x="81.28" y="68.58"/>
 <instance part="GND26" gate="1" x="81.28" y="60.96"/>
@@
 <instance part="GND30" gate="1" x="170.18" y="60.96"/>
 <instance part="SUPPLY1" gate="1" x="81.28" y="106.68"/>
+<instance part="D2" gate="G$1" x="104.14" y="93.98" rot="R180"/>
 </instances>
 <busses>
@@
 <pinref part="GND24" gate="1" pin="GND"/>
 <wire x1="144.78" y1="66.04" x2="144.78" y2="63.5" width="0.1524" layer="91"/>
-</segment>
-<segment>
-<pinref part="Q3" gate="G$1" pin="C"/>
-<pinref part="GND25" gate="1" pin="GND"/>
-<wire x1="132.08" y1="66.04" x2="132.08" y2="63.5" width="0.1524" layer="91"/>
 </segment>
 <segment>
@@
 <wire x1="124.46" y1="93.98" x2="114.3" y2="93.98" width="0.1524" layer="91"/>
 <wire x1="114.3" y1="93.98" x2="114.3" y2="91.44" width="0.1524" layer="91"/>
-<pinref part="D3" gate="1" pin="A"/>
 <wire x1="114.3" y1="93.98" x2="106.68" y2="93.98" width="0.1524" layer="91"/>
 <junction x="114.3" y="93.98"/>
-</segment>
-</net>
-<net name="N$11" class="0">
-<segment>
+<pinref part="D2" gate="G$1" pin="A"/>
+</segment>
+</net>
+<net name="N$16" class="0">
+<segment>
+<pinref part="Q2" gate="G$1" pin="G"/>
+<wire x1="106.68" y1="83.82" x2="109.22" y2="83.82" width="0.1524" layer="91"/>
+<wire x1="106.68" y1="81.28" x2="106.68" y2="83.82" width="0.1524" layer="91"/>
+<wire x1="144.78" y1="81.28" x2="106.68" y2="81.28" width="0.1524" layer="91"/>
 <pinref part="U$6" gate="G$1" pin="SWE"/>
 <pinref part="R11" gate="G$1" pin="1"/>
 <wire x1="172.72" y1="88.9" x2="144.78" y2="88.9" width="0.1524" layer="91"/>
 <wire x1="144.78" y1="88.9" x2="144.78" y2="81.28" width="0.1524" layer="91"/>
-<pinref part="D2" gate="G$1" pin="A"/>
-<wire x1="144.78" y1="81.28" x2="144.78" y2="78.74" width="0.1524" layer="91"/>
-<wire x1="144.78" y1="78.74" x2="144.78" y2="76.2" width="0.1524" layer="91"/>
-<wire x1="139.7" y1="81.28" x2="144.78" y2="81.28" width="0.1524" layer="91"/>
-<pinref part="Q3" gate="G$1" pin="B"/>
-<wire x1="127" y1="71.12" x2="127" y2="78.74" width="0.1524" layer="91"/>
-<wire x1="127" y1="78.74" x2="144.78" y2="78.74" width="0.1524" layer="91"/>
+<wire x1="144.78" y1="81.28" x2="144.78" y2="76.2" width="0.1524" layer="91"/>
 <junction x="144.78" y="81.28"/>
-<junction x="144.78" y="78.74"/>
-</segment>
-</net>
-<net name="N$16" class="0">
-<segment>
-<pinref part="Q2" gate="G$1" pin="G"/>
-<wire x1="106.68" y1="83.82" x2="109.22" y2="83.82" width="0.1524" layer="91"/>
-<wire x1="106.68" y1="81.28" x2="106.68" y2="83.82" width="0.1524" layer="91"/>
-<pinref part="D2" gate="G$1" pin="C"/>
-<wire x1="134.62" y1="81.28" x2="132.08" y2="81.28" width="0.1524" layer="91"/>
-<pinref part="Q3" gate="G$1" pin="E"/>
-<wire x1="132.08" y1="81.28" x2="106.68" y2="81.28" width="0.1524" layer="91"/>
-<wire x1="132.08" y1="76.2" x2="132.08" y2="81.28" width="0.1524" layer="91"/>
-<junction x="132.08" y="81.28"/>
 </segment>
 </net>
@@
 <net name="V+" class="0">
 <segment>
-<pinref part="D3" gate="1" pin="C"/>
 <wire x1="101.6" y1="93.98" x2="91.44" y2="93.98" width="0.1524" layer="91"/>
 <pinref part="C13" gate="G$1" pin="+"/>
@@
 <junction x="81.28" y="93.98"/>
 <junction x="91.44" y="93.98"/>
-</segment>
-</net>
+<pinref part="D2" gate="G$1" pin="C"/>
+</segment>
+</net>
